File: hardware/jotakey-key/jotakey-key.kicad_pcb (KiCad board)
At the start: 2 copper layers, 18 x 45.5 mm, 27 parts, among them J1 USB_A_PCB_Edge, U1 STM32L432KCU6, U2 SLS32AIA010MH, U3 XC6206P332MR, U4 USBLC6-2SC6

Commit message: hardware: version the board as HW 0.1.0
The hardware version lives in one place, the KiCad project text variable
HW_VERSION. The schematic and PCB title blocks and a new "HW x.y.z" text
on the bottom silkscreen, behind the touch electrode, all show
${HW_VERSION}. HARDWARE.md describes the scheme: hardware tags
hw-vX.Y.Z, firmware tags fw-vX.Y.Z.

tools/silk.py now updates its items in place instead of removing and
re-adding them, which the KiCad 10 bindings do not survive.

Co-Authored-By: Claude Opus 5.5 <noreply@anthropic.com>
Other:
- board text added: "HW ${HW_VERSION}"
Changed lines of the file:
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@@
 	)
 	(paper "A4")
+	(title_block
+		(title "Jotakey key: STM32L432 + OPTIGA Trust M USB-A dongle")
+		(date "2026-10-17")
+		(rev "${HW_VERSION}")
+		(company "Jotakey")
+		(comment 1 "Pin plan and parts: hardware/HARDWARE.md")
+		(comment 2 "Fabrication and assembly: JLCPCB, 2 layers, 2.0 mm, ENIG")
+	)
 	(layers
 		(0 "F.Cu" signal)
@@
 		)
 	)
+	(property "HW_VERSION" "0.1.0")
 	(footprint "Resistor_SMD:R_0402_1005Metric"
 		(layer "F.Cu")
@@
 		(layer "Edge.Cuts")
 	)
+	(gr_text "HW ${HW_VERSION}"
+		(at 100 106.5 0)
+		(layer "B.SilkS")
+		(effects
+			(font
+				(size 1 1)
+				(thickness 0.15)
+			)
+			(justify mirror)
+		)
+	)
 	(segment

Commit message: hardware: mark where JLCPCB prints the order number
"JLCJLCJLCJLC" on the bottom silkscreen, along the long edge opposite the
serial-number block, 0.8 mm high (JLCPCB's minimum). Order with "Remove
order number: specify a location" for JLCPCB to print it there.

Co-Authored-By: Claude Opus 5.5 <noreply@anthropic.com>
Other:
- board text added: "JLCJLCJLCJLC"
Changed lines of the file:
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@@
 		(layer "Edge.Cuts")
+	)
+	(gr_text "JLCJLCJLCJLC"
+		(at 107.6 97 90)
+		(layer "B.SilkS")
+		(effects
+			(font
+				(size 0.8 0.8)
+				(thickness 0.15)
+			)
+			(justify mirror)
+		)
 	)
 	(gr_text "HW ${HW_VERSION}"
